Commit message: Remove collision for dishwasher tray
because it's too heavy to load in bullet.

File: iai_apartment/urdf/kitchen_unreal.xacro (robot description, xacro)
@@ -2686,9 +2686,9 @@
         </geometry>
       </visual>
-      <collision>
+<!--       <collision>
         <geometry>
           <mesh filename="package://iai_apartment/meshes/unreal/SM_Dishwasher_Tray_01.stl" />
         </geometry>
-      </collision>
+      </collision> -->
     </link>
     <joint name="dishwasher_tray2_joint" type="prismatic">
@@ -2705,9 +2705,9 @@
         </geometry>
       </visual>
-      <collision>
+<!--       <collision>
         <geometry>
           <mesh filename="package://iai_apartment/meshes/unreal/SM_Dishwasher_Tray_02.stl" />
         </geometry>
-      </collision>
+      </collision> -->
     </link>
     <joint name="dishwasher_tray3_joint" type="prismatic">
@@ -2724,9 +2724,9 @@
         </geometry>
       </visual>
-      <collision>
+<!--       <collision>
         <geometry>
           <mesh filename="package://iai_apartment/meshes/unreal/SM_Dishwasher_Tray_03.stl" />
         </geometry>
-      </collision>
+      </collision> -->
     </link>
     <!-- Cabinet8 -->
